File: USB_switch.kicad_sch (KiCad schematic)
At the start: 4 parts, among them U4 TS3USB30EDGSR, U5 AMS1117-3.3

Commit message: Change voltage value
Connections:
- net +5V renamed +5V standby
Changed lines of the file:
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@@
 			)
 		)
-		(property "Value" "+5V"
+		(property "Value" "+5V standby"
 			(at 46.99 38.1 0)
 			(effects

Commit message: Fix USB connection
Connections:
- net USB_DIN.D+ renamed USB_DIN.+
- net USB_DIN.D- renamed USB_DIN.-
- net USB_RJ.D+ renamed USB_RJ.+
- net USB_RJ.D- renamed USB_RJ.-
- net USB_port.D+ renamed USB_port.+
- net USB_port.D- renamed USB_port.-
